File: plate/plate.kicad_pcb (KiCad board)
At the start: 2 copper layers, 313.9 x 116.5 mm, 0 parts

Commit message: upd
Routing:
- added copper zone on B.Cu, net GND
- added copper zone on F.Cu, net GND
Other:
- board size 313.9 x 116.5 mm -> 338.1 x 116.2 mm
- board text added: "12"
- board text added: "ア ユ ム"
